File: Reciever/Reciever.kicad_sch (KiCad schematic)
At the start: 8 parts, among them J1 Conn_01x01_Socket, J2 Conn_01x02_Socket, J3 Conn_01x02_Socket, U2 LM393BIPWR, U3 LM386MX-1_NOPB

Commit message: updated to utilise more common parts
Parts:
- removed C2: 0603YC104KAZ2A, 0603YC104KAZ2A:CAPC1608X90N, symbol 0603YC104KAZ2A:0603YC104KAZ2A
- removed R2: PVG3G103C01R00, PVG3G103C01R00:TRIM_PVG3G103C01R00, symbol PVG3G103C01R00:PVG3G103C01R00
- removed R3: CR0603AFX-1002EAS, CR0603AFX-1002EAS:RESC1608X55N, symbol CR0603AFX-1002EAS:CR0603AFX-1002EAS
- added C1: CL31B104KBCNNNC, CL31B104KBCNNNC:CAPC3216X100N, symbol CL31B104KBCNNNC:CL31B104KBCNNNC
- added R1: 1206W4F1002T5E, 1206W4F1002T5E:RESC3115X65N, symbol 1206W4F1002T5E:1206W4F1002T5E
- added VR1: 3314J-1-100E, 3314J-1-100E:TRIM_3314J-1-100E, symbol 3314J-1-100E:3314J-1-100E
- J1, J2, J3: now left out of the parts list
- renumbered U3 to U1
Connections:
- net +5V: now also VR1.1
- net GND: now also R1.2, VR1.3
- net at J2.1 (Pin_1): now also C1.1, R1.1
- net at U1.3 (+INPUT): now also C1.2
- net at U2.3: now also VR1.2

Commit message: Added images to the readme
Parts:
- J2: value Conn_01x02_Socket -> Piezo pins
- J3: value Conn_01x02_Socket -> Board Power
Other:
- moved on the sheet: J1
Changed lines of the file:
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@@
 	(wire
 		(pts
-			(xy 163.83 66.04) (xy 173.99 66.04)
+			(xy 163.83 66.04) (xy 165.1 66.04)
 		)
 		(stroke
@@
 			)
 		)
-		(property "Value" "Conn_01x02_Socket"
+		(property "Value" "Piezo pins"
 			(at 34.925 50.8 0)
 			(effects
@@
 			)
 		)
-		(property "Value" "Conn_01x02_Socket"
+		(property "Value" "Board Power"
 			(at 25.4 67.3099 0)
 			(effects
@@
 		(on_board yes)
 		(dnp no)
-		(fields_autoplaced yes)
 		(property "Reference" "U2"
-			(at 166.37 59.9692 0)
+			(at 146.558 73.914 0)
 			(effects
 				(font
@@
 		)
 		(property "Value" "LM393BIPWR"
-			(at 166.37 62.5092 0)
+			(at 146.558 76.454 0)
 			(effects
 				(font
@@
 	(symbol
 		(lib_id "Connector:Conn_01x01_Socket")
-		(at 179.07 66.04 0)
+		(at 170.18 66.04 0)
 		(unit 1)
 		(exclude_from_sim no)
@@
 		(fields_autoplaced yes)
 		(property "Reference" "J1"
-			(at 180.34 64.7699 0)
+			(at 171.45 64.7699 0)
 			(effects
 				(font
@@
 		)
 		(property "Value" "Conn_01x01_Socket"
-			(at 180.34 67.3099 0)
+			(at 171.45 67.3099 0)
 			(effects
 				(font
@@
 		)
 		(property "Footprint" "Connector_Wire:SolderWire-0.1sqmm_1x01_D0.4mm_OD1mm"
-			(at 179.07 66.04 0)
+			(at 170.18 66.04 0)
 			(effects
 				(font
@@
 		)
 		(property "Datasheet" "~"
-			(at 179.07 66.04 0)
+			(at 170.18 66.04 0)
 			(effects
 				(font
@@
 		)
 		(property "Description" "Generic connector, single row, 01x01, script generated"
-			(at 179.07 66.04 0)
-			(effects
-				(font
+			(at 170.18 66.04 0)
+			(effects
+				(font

Commit message: Updated to add resistor pad for gain, and 5v flood to CL2
Parts:
- added R2: 1206W4F1002T5E, 1206W4F1002T5E:RESC3115X65N, symbol 1206W4F1002T5E:1206W4F1002T5E
Connections:
- net at U1.1 (GAIN): now also R2.1; no longer U1.8 (GAIN)
- new net: R2.2, U1.8 (GAIN)
